Commit message: Gazebo simulator added - empty world + Mr. Peterbot

File: src/mr_peterbot_description/urdf/mr_peterbot.urdf.xacro (robot description, xacro)
@@ -148,3 +148,46 @@
         <origin xyz="${chassis_length/2} 0 0"/>
     </joint>
+    <!-- === GAZEBO SIMULATION SETUP === -->
+     <!-- ===== GAZEBO MATERIALS ===== -->
+    <gazebo reference="chassis">
+        <material>Gazebo/Blue</material>
+    </gazebo>
+    <gazebo reference="lidar_link">
+        <material>Gazebo/Black</material>
+    </gazebo>
+    <gazebo reference="camera_link">
+        <material>Gazebo/Red</material>
+    </gazebo>
+    <gazebo reference="front_left_wheel">
+        <material>Gazebo/Black</material>
+        <mu1>0.8</mu1>
+        <mu2>0.8</mu2>
+    </gazebo>
+    <gazebo reference="front_right_wheel">
+        <material>Gazebo/Black</material>
+        <mu1>0.8</mu1>
+        <mu2>0.8</mu2>
+    </gazebo>
+    <gazebo reference="rear_left_wheel">
+        <material>Gazebo/Black</material>
+        <mu1>0.8</mu1>
+        <mu2>0.8</mu2>
+    </gazebo>
+    <gazebo reference="rear_right_wheel">
+        <material>Gazebo/Black</material>
+        <mu1>0.8</mu1>
+        <mu2>0.8</mu2>
+    </gazebo>
+    <!-- ===== GAZEBO PHYSICS PLUGIN ===== -->
+    <gazebo>
+    <plugin filename="gz-sim-diff-drive-system"
+            name="gz::sim::systems::DiffDrive">
+        <left_joint>rear_left_wheel_joint</left_joint>
+        <right_joint>rear_right_wheel_joint</right_joint>
+        <wheel_separation>${wheel_y_offset * 2}</wheel_separation>
+        <wheel_radius>${wheel_radius}</wheel_radius>
+        <odom_publish_frequency>10</odom_publish_frequency>
+        <topic>cmd_vel</topic>
+    </plugin>
+    </gazebo>
 </robot>

Commit message: ros2_control added - Moves in Gazebo

File: src/mr_peterbot_description/urdf/mr_peterbot.urdf.xacro (robot description, xacro)
@@ -179,15 +179,36 @@
         <mu2>0.8</mu2>
     </gazebo>
-    <!-- ===== GAZEBO PHYSICS PLUGIN ===== -->
+    <!-- ===== ROS2 CONTROL ===== -->
+    <ros2_control name="mr_peterbot" type="system">
+        <hardware>
+        <plugin>gz_ros2_control/GazeboSimSystem</plugin>
+        </hardware>
+        <!-- Back wheels — Actibves -->
+        <joint name="rear_left_wheel_joint">
+        <command_interface name="velocity"/>
+        <state_interface name="velocity"/>
+        <state_interface name="position"/>
+        </joint>
+        <joint name="rear_right_wheel_joint">
+        <command_interface name="velocity"/>
+        <state_interface name="velocity"/>
+        <state_interface name="position"/>
+        </joint>
+        <!-- Front Wheels — sPassives -->
+        <joint name="front_left_wheel_joint">
+        <state_interface name="velocity"/>
+        <state_interface name="position"/>
+        </joint>
+        <joint name="front_right_wheel_joint">
+        <state_interface name="velocity"/>
+        <state_interface name="position"/>
+        </joint>
+    </ros2_control>
+    <!-- ===== GZ ROS2 CONTROL PLUGIN ===== -->
     <gazebo>
-    <plugin filename="gz-sim-diff-drive-system"
-            name="gz::sim::systems::DiffDrive">
-        <left_joint>rear_left_wheel_joint</left_joint>
-        <right_joint>rear_right_wheel_joint</right_joint>
-        <wheel_separation>${wheel_y_offset * 2}</wheel_separation>
-        <wheel_radius>${wheel_radius}</wheel_radius>
-        <odom_publish_frequency>10</odom_publish_frequency>
-        <topic>cmd_vel</topic>
-    </plugin>
+        <plugin filename="gz_ros2_control-system"
+                name="gz_ros2_control::GazeboSimROS2ControlPlugin">
+        <parameters>$(find mr_peterbot_bringup)/config/controllers.yaml</parameters>
+        </plugin>
     </gazebo>
 </robot>

Commit message: Neighborhood added - The Village OKC

File: src/mr_peterbot_description/urdf/mr_peterbot.urdf.xacro (robot description, xacro)
@@ -63,5 +63,6 @@
         <parent link="base_link"/>
         <child  link="chassis"/>
-        <origin xyz="0 0 ${wheel_radius + chassis_height/2}"/>
+        <origin xyz="0 0 ${wheel_radius + chassis_height/2}"
+          rpy="0 0 3.1416"/>
     </joint>
     <!-- ===== WHEEL MACRO ===== -->
@@ -93,8 +94,8 @@
     </xacro:macro>
     <!-- ===== ADDIND THE 4 WHEELS ===== -->
-    <xacro:wheel name="front_left"  x=" ${wheel_x_offset}" y=" ${wheel_y_offset}"/>
-    <xacro:wheel name="front_right" x=" ${wheel_x_offset}" y="-${wheel_y_offset}"/>
-    <xacro:wheel name="rear_left"   x="-${wheel_x_offset}" y=" ${wheel_y_offset}"/>
-    <xacro:wheel name="rear_right"  x="-${wheel_x_offset}" y="-${wheel_y_offset}"/>
+    <xacro:wheel name="front_left"  x="-${wheel_x_offset}" y=" ${wheel_y_offset}"/>
+    <xacro:wheel name="front_right" x="-${wheel_x_offset}" y="-${wheel_y_offset}"/>
+    <xacro:wheel name="rear_left"   x=" ${wheel_x_offset}" y=" ${wheel_y_offset}"/>
+    <xacro:wheel name="rear_right"  x=" ${wheel_x_offset}" y="-${wheel_y_offset}"/>
     <!-- ===== LiDAR ===== -->
     <link name="lidar_link">

Commit message: Ackermann sterring add and control modified

File: src/mr_peterbot_description/urdf/mr_peterbot.urdf.xacro (robot description, xacro)
@@ -2,9 +2,10 @@
 <robot xmlns:xacro="http://www.ros.org/wiki/xacro" name="mr_peterbot">
     <!-- === VARIABLES ===-->
-    <!-- CAR DIMENSIONS -->
+    <!-- MAIN BODY -->
     <xacro:property name="chassis_length" value="0.4"/>
     <xacro:property name="chassis_width"  value="0.2"/>
     <xacro:property name="chassis_height" value="0.1"/>
     <xacro:property name="chassis_mass"   value="2.0"/>
+    <!-- WHEELS -->
     <xacro:property name="wheel_radius"   value="0.05"/>
     <xacro:property name="wheel_width"    value="0.04"/>
@@ -12,20 +13,39 @@
     <xacro:property name="wheel_x_offset" value="0.13"/>
     <xacro:property name="wheel_y_offset" value="0.12"/>
-    <!-- LiDAR DIMENSIONS -->
-    <xacro:property name="lidar_radius" value="0.04"/>
-    <xacro:property name="lidar_height" value="0.06"/>
-    <xacro:property name="lidar_mass"   value="0.1"/>
-    <!-- Camera DIMENSIONS -->
+    <!-- CINEMATIC AND DYNAMICS VALUES-->
+    <xacro:property name="max_steering_angle"            value="0.6108652"/>
+    <xacro:property name="max_steering_angular_velocity" value="1.570796"/>
+    <xacro:property name="max_steering_effort"           value="1.0"/>
+    <xacro:property name="max_velocity"                  value="2.0"/>
+    <xacro:property name="max_effort"                    value="10.0"/>
+    <xacro:property name="max_wheel_angular_velocity"    value="${max_velocity / wheel_radius}"/>
+    <!-- LiDAR -->
+    <xacro:property name="lidar_radius"      value="0.04"/>
+    <xacro:property name="lidar_height"      value="0.06"/>
+    <xacro:property name="lidar_mass"        value="0.1"/>
+    <xacro:property name="lidar_min_angle"   value="-3.14159"/>
+    <xacro:property name="lidar_max_angle"   value="3.14159"/>
+    <xacro:property name="lidar_samples"     value="360"/>
+    <xacro:property name="lidar_min_range"   value="0.12"/>
+    <xacro:property name="lidar_max_range"   value="50"/>
+    <xacro:property name="lidar_update_rate" value="10.0"/>
+    <xacro:property name="lidar_noise_mean"   value="0.0"/>
+    <xacro:property name="lidar_noise_stddev" value="0.01"/>
+    <!-- CAMERA -->
     <xacro:property name="camera_width"  value="0.05"/>
     <xacro:property name="camera_height" value="0.03"/>
     <xacro:property name="camera_depth"  value="0.03"/>
     <xacro:property name="camera_mass"   value="0.05"/>
-    <!-- ===== INERTIA MACROS (CHASIS AND WHEELS) ===== -->
+    <xacro:property name="camera_fov"    value="1.3962634"/>
+    <xacro:property name="camera_fps"    value="30"/>
+    <xacro:property name="image_width"   value="640"/>
+    <xacro:property name="image_height"  value="480"/>
+    <!-- ===== INERTIA MACROS ===== -->
     <xacro:macro name="box_inertia" params="m l w h">
         <inertial>
             <mass value="${m}"/>
             <inertia ixx="${(1/12) * m * (w*w + h*h)}" ixy="0.0" ixz="0.0"
-                    iyy="${(1/12) * m * (l*l + h*h)}" iyz="0.0"
-                    izz="${(1/12) * m * (l*l + w*w)}"/>
+                     iyy="${(1/12) * m * (l*l + h*h)}" iyz="0.0"
+                     izz="${(1/12) * m * (l*l + w*w)}"/>
         </inertial>
     </xacro:macro>
@@ -34,19 +54,19 @@
             <mass value="${m}"/>
             <inertia ixx="${(1/12) * m * (3*r*r + l*l)}" ixy="0.0" ixz="0.0"
-                    iyy="${(1/12) * m * (3*r*r + l*l)}" iyz="0.0"
-                    izz="${(1/2)  * m * r*r}"/>
-            </inertial>
+                     iyy="${(1/12) * m * (3*r*r + l*l)}" iyz="0.0"
+                     izz="${(1/2)  * m * r*r}"/>
+        </inertial>
     </xacro:macro>
     <!-- ===== BASE LINK ===== -->
     <link name="base_link"/>
-    <!-- ===== CHASSIS OF MR. PETERBOT RC CAR ===== -->
+    <!-- ===== CHASSIS ===== -->
     <link name="chassis">
         <visual>
             <geometry>
                 <box size="${chassis_length} ${chassis_width} ${chassis_height}"/>
-        </geometry>
-        <material name="blue">
-            <color rgba="0.0 0.0 0.8 1.0"/>
-        </material>
+            </geometry>
+            <material name="blue">
+                <color rgba="0.0 0.0 0.8 1.0"/>
+            </material>
         </visual>
         <collision>
@@ -56,18 +76,19 @@
         </collision>
         <xacro:box_inertia m="${chassis_mass}"
-                       l="${chassis_length}"
-                       w="${chassis_width}"
-                       h="${chassis_height}"/>
+                           l="${chassis_length}"
+                           w="${chassis_width}"
+                           h="${chassis_height}"/>
     </link>
     <joint name="base_to_chassis" type="fixed">
         <parent link="base_link"/>
         <child  link="chassis"/>
-        <origin xyz="0 0 ${wheel_radius + chassis_height/2}"
-          rpy="0 0 3.1416"/>
+        <origin xyz="0 0 ${wheel_radius + chassis_height/2}" rpy="0 0 3.1416"/>
     </joint>
-    <!-- ===== WHEEL MACRO ===== -->
-    <xacro:macro name="wheel" params="name x y">
-        <link name="${name}_wheel">
+    <!-- ===== WHEEL MACROS ===== -->
+    <!-- FRONT WHEEL MACRO = WHEEL LINK + STEERING LINK -->
+    <xacro:macro name="front_wheel" params="prefix">
+        <link name="${prefix}_wheel_link">
             <visual>
+                <origin xyz="0.0 0.0 0.0" rpy="0 0 0"/>
                 <geometry>
                     <cylinder radius="${wheel_radius}" length="${wheel_width}"/>
@@ -78,30 +99,100 @@
             </visual>
             <collision>
+                <origin xyz="0.0 0.0 0.0" rpy="0 0 0"/>
                 <geometry>
                     <cylinder radius="${wheel_radius}" length="${wheel_width}"/>
                 </geometry>
             </collision>
-            <xacro:cylinder_inertia m="${wheel_mass}"
-                               r="${wheel_radius}"
-                               l="${wheel_width}"/>
+            <xacro:cylinder_inertia m="${wheel_mass}" r="${wheel_radius}" l="${wheel_width}"/>
         </link>
-        <joint name="${name}_wheel_joint" type="continuous">
+        <link name="${prefix}_steering_link">
+            <visual>
+                <origin xyz="0.0 0.0 0.0" rpy="0 0 0"/>
+                <geometry>
+                    <cylinder length="0.001" radius="0.01"/>
+                </geometry>
+            </visual>
+            <collision>
+                <origin xyz="0.0 0.0 0.0" rpy="0 0 0"/>
+                <geometry>
+                    <cylinder length="0.001" radius="0.01"/>
+                </geometry>
+            </collision>
+            <inertial>
+                <mass value="0.01"/>
+                <inertia ixx="1e-6" ixy="0.0" ixz="0.0"
+                         iyy="1e-6" iyz="0.0"
+                         izz="1e-6"/>
+            </inertial>
+        </link>
+    </xacro:macro>
+    <!-- REAR WHEEL MACRO = WHEEL LINK ONLY -->
+    <xacro:macro name="rear_wheel" params="prefix">
+        <link name="${prefix}_wheel_link">
+            <visual>
+                <origin xyz="0.0 0.0 0.0" rpy="0 0 0"/>
+                <geometry>
+                    <cylinder radius="${wheel_radius}" length="${wheel_width}"/>
+                </geometry>
+                <material name="black">
+                    <color rgba="0.1 0.1 0.1 1.0"/>
+                </material>
+            </visual>
+            <collision>
+                <origin xyz="0.0 0.0 0.0" rpy="0 0 0"/>
+                <geometry>
+                    <cylinder radius="${wheel_radius}" length="${wheel_width}"/>
+                </geometry>
+            </collision>
+            <xacro:cylinder_inertia m="${wheel_mass}" r="${wheel_radius}" l="${wheel_width}"/>
+        </link>
+    </xacro:macro>
+    <!-- ===== CREATING THE 4 WHEELS ===== -->
+    <xacro:front_wheel prefix="front_left"/>
+    <xacro:front_wheel prefix="front_right"/>
+    <xacro:rear_wheel  prefix="rear_left"/>
+    <xacro:rear_wheel  prefix="rear_right"/>
+    <!-- ===== JOINT MACROS ===== -->
+    <!-- FRONT WHEEL JOINTS: steering (revolute) + wheel (continuous) -->
+    <xacro:macro name="front_wheel_joints" params="prefix x y">
+        <joint name="${prefix}_steering_joint" type="revolute">
+            <origin xyz="${x} ${y} -${wheel_radius/2}" rpy="0 0 0"/>
             <parent link="chassis"/>
-            <child  link="${name}_wheel"/>
-            <origin xyz="${x} ${y} 0" rpy="${pi/2} 0 0"/>
+            <child link="${prefix}_steering_link"/>
             <axis xyz="0 0 1"/>
-        </joint>
-    </xacro:macro>
-    <!-- ===== ADDIND THE 4 WHEELS ===== -->
-    <xacro:wheel name="front_left"  x="-${wheel_x_offset}" y=" ${wheel_y_offset}"/>
-    <xacro:wheel name="front_right" x="-${wheel_x_offset}" y="-${wheel_y_offset}"/>
-    <xacro:wheel name="rear_left"   x=" ${wheel_x_offset}" y=" ${wheel_y_offset}"/>
-    <xacro:wheel name="rear_right"  x=" ${wheel_x_offset}" y="-${wheel_y_offset}"/>
+            <limit effort="${max_steering_effort}"
+                   lower="${-max_steering_angle}"
+                   upper="${max_steering_angle}"
+                   velocity="${max_steering_angular_velocity}"/>
+            <dynamics damping="0.1" friction="0.1"/>
+        </joint>
+        <joint name="${prefix}_wheel_joint" type="continuous">
+            <origin xyz="0 0 0" rpy="1.5708 0 0"/>
+            <parent link="${prefix}_steering_link"/>
+            <child link="${prefix}_wheel_link"/>
+            <axis xyz="0 0 1"/>
+            <dynamics damping="0.1" friction="0.1"/>
+        </joint>
+    </xacro:macro>
+    <!-- REAR WHEEL JOINT: wheel only (continuous) -->
+    <xacro:macro name="rear_wheel_joint" params="prefix x y">
+        <joint name="${prefix}_wheel_joint" type="continuous">
+            <origin xyz="${x} ${y} -${wheel_radius/2}" rpy="1.5708 0 0"/>
+            <parent link="chassis"/>
+            <child link="${prefix}_wheel_link"/>
+            <axis xyz="0 0 1"/>
+            <dynamics damping="0.1" friction="0.1"/>
+        </joint>
+    </xacro:macro>
+    <!-- ===== CREATING THE JOINTS FOR EACH WHEEL ===== -->
+    <xacro:front_wheel_joints prefix="front_left"  x=" ${wheel_x_offset}" y=" ${wheel_y_offset}"/>
+    <xacro:front_wheel_joints prefix="front_right" x=" ${wheel_x_offset}" y="-${wheel_y_offset}"/>
+    <xacro:rear_wheel_joint   prefix="rear_left"   x="-${wheel_x_offset}" y=" ${wheel_y_offset}"/>
+    <xacro:rear_wheel_joint   prefix="rear_right"  x="-${wheel_x_offset}" y="-${wheel_y_offset}"/>
     <!-- ===== LiDAR ===== -->
     <link name="lidar_link">
         <visual>
             <geometry>
-                <cylinder radius="${lidar_radius}"
-                        length="${lidar_height}"/>
+                <cylinder radius="${lidar_radius}" length="${lidar_height}"/>
             </geometry>
             <material name="black">
@@ -111,11 +202,8 @@
         <collision>
             <geometry>
-                <cylinder radius="${lidar_radius}"
-                        length="${lidar_height}"/>
+                <cylinder radius="${lidar_radius}" length="${lidar_height}"/>
             </geometry>
         </collision>
-        <xacro:cylinder_inertia m="${lidar_mass}"
-                                r="${lidar_radius}"
-                                l="${lidar_height}"/>
+        <xacro:cylinder_inertia m="${lidar_mass}" r="${lidar_radius}" l="${lidar_height}"/>
     </link>
     <joint name="lidar_joint" type="fixed">
@@ -140,76 +228,107 @@
         </collision>
         <xacro:box_inertia m="${camera_mass}"
-                        l="${camera_depth}"
-                        w="${camera_width}"
-                        h="${camera_height}"/>
+                           l="${camera_depth}"
+                           w="${camera_width}"
+                           h="${camera_height}"/>
     </link>
     <joint name="camera_joint" type="fixed">
         <parent link="chassis"/>
         <child  link="camera_link"/>
-        <origin xyz="${chassis_length/2} 0 0"/>
+        <origin xyz="${chassis_length/2 + camera_depth/2} 0 ${chassis_height/2}"/>
     </joint>
-    <!-- === GAZEBO SIMULATION SETUP === -->
-     <!-- ===== GAZEBO MATERIALS ===== -->
+    <!-- ===== GAZEBO SIMULATION SETUP ===== -->
     <gazebo reference="chassis">
         <material>Gazebo/Blue</material>
+        <mu1>0.001</mu1>
+        <mu2>0.001</mu2>
+    </gazebo>
+    <gazebo reference="front_left_wheel_link">
+        <mu1>0.8</mu1>
+        <mu2>0.8</mu2>
+    </gazebo>
+    <gazebo reference="front_right_wheel_link">
+        <mu1>0.8</mu1>
+        <mu2>0.8</mu2>
+    </gazebo>
+    <gazebo reference="rear_left_wheel_link">
+        <mu1>0.8</mu1>
+        <mu2>0.8</mu2>
+    </gazebo>
+    <gazebo reference="rear_right_wheel_link">
+        <mu1>0.8</mu1>
+        <mu2>0.8</mu2>
     </gazebo>
     <gazebo reference="lidar_link">
         <material>Gazebo/Black</material>
+        <mu1>0.001</mu1>
+        <mu2>0.001</mu2>
     </gazebo>
     <gazebo reference="camera_link">
         <material>Gazebo/Red</material>
-    </gazebo>
-    <gazebo reference="front_left_wheel">
-        <material>Gazebo/Black</material>
-        <mu1>0.8</mu1>
-        <mu2>0.8</mu2>
-    </gazebo>
-    <gazebo reference="front_right_wheel">
-        <material>Gazebo/Black</material>
-        <mu1>0.8</mu1>
-        <mu2>0.8</mu2>
-    </gazebo>
-    <gazebo reference="rear_left_wheel">
-        <material>Gazebo/Black</material>
-        <mu1>0.8</mu1>
-        <mu2>0.8</mu2>
-    </gazebo>
-    <gazebo reference="rear_right_wheel">
-        <material>Gazebo/Black</material>
-        <mu1>0.8</mu1>
-        <mu2>0.8</mu2>
+        <mu1>0.001</mu1>
+        <mu2>0.001</mu2>
     </gazebo>
     <!-- ===== ROS2 CONTROL ===== -->
     <ros2_control name="mr_peterbot" type="system">
         <hardware>
-        <plugin>gz_ros2_control/GazeboSimSystem</plugin>
+            <plugin>gz_ros2_control/GazeboSimSystem</plugin>
         </hardware>
-        <!-- Back wheels — Actibves -->
+        <joint name="front_left_steering_joint">
+            <command_interface name="position">
+                <param name="min">${-max_steering_angle}</param>
+                <param name="max">${max_steering_angle}</param>
+            </command_interface>
+            <state_interface name="position"/>
+            <state_interface name="velocity"/>
+            <state_interface name="effort"/>
+        </joint>
+        <joint name="front_right_steering_joint">
+            <command_interface name="position">
+                <param name="min">${-max_steering_angle}</param>
+                <param name="max">${max_steering_angle}</param>
+            </command_interface>
+            <state_interface name="position"/>
+            <state_interface name="velocity"/>
+            <state_interface name="effort"/>
+        </joint>
         <joint name="rear_left_wheel_joint">
-        <command_interface name="velocity"/>
-        <state_interface name="velocity"/>
-        <state_interface name="position"/>
+            <command_interface name="velocity">
+                <param name="min">${-max_wheel_angular_velocity}</param>
+                <param name="max">${max_wheel_angular_velocity}</param>
+            </command_interface>
+            <state_interface name="position"/>
+            <state_interface name="velocity"/>
+            <state_interface name="effort"/>
         </joint>
         <joint name="rear_right_wheel_joint">
-        <command_interface name="velocity"/>
-        <state_interface name="velocity"/>
-        <state_interface name="position"/>
-        </joint>
-        <!-- Front Wheels — sPassives -->
-        <joint name="front_left_wheel_joint">
-        <state_interface name="velocity"/>
-        <state_interface name="position"/>
-        </joint>
-        <joint name="front_right_wheel_joint">
-        <state_interface name="velocity"/>
-        <state_interface name="position"/>
+            <command_interface name="velocity">
+                <param name="min">${-max_wheel_angular_velocity}</param>
+                <param name="max">${max_wheel_angular_velocity}</param>
+            </command_interface>
+            <state_interface name="position"/>
+            <state_interface name="velocity"/>
+            <state_interface name="effort"/>
         </joint>
     </ros2_control>
-    <!-- ===== GZ ROS2 CONTROL PLUGIN ===== -->
+    <!-- ===== GAZEBO PLUGINS ===== -->
     <gazebo>
+        <plugin filename="gz-sim-joint-state-publisher-system"
+                name="gz::sim::systems::JointStatePublisher">
+            <topic>joint_states</topic>
+            <joint_name>front_left_steering_joint</joint_name>
+            <joint_name>front_right_steering_joint</joint_name>
+            <joint_name>front_left_wheel_joint</joint_name>
+            <joint_name>front_right_wheel_joint</joint_name>
+            <joint_name>rear_left_wheel_joint</joint_name>
+            <joint_name>rear_right_wheel_joint</joint_name>
+        </plugin>
         <plugin filename="gz_ros2_control-system"
                 name="gz_ros2_control::GazeboSimROS2ControlPlugin">
-        <parameters>$(find mr_peterbot_bringup)/config/controllers.yaml</parameters>
+            <parameters>$(find mr_peterbot_bringup)/config/controllers.yaml</parameters>
         </plugin>
+        <plugin filename="gz-sim-sensors-system"
+                name="gz::sim::systems::Sensors">
+            <render_engine>ogre2</render_engine>
+        </plugin>
     </gazebo>
 </robot>
