Commit message: Ackermann stering added to Mr. Peterbot and simulated with a C++ control node

File: src/mr_peterbot_description/urdf/mr_peterbot.urdf.xacro (robot description, xacro)
@@ -16,5 +16,5 @@
     <xacro:property name="max_steering_angle"            value="0.6108652"/>
     <xacro:property name="max_steering_angular_velocity" value="1.570796"/>
-    <xacro:property name="max_steering_effort"           value="1.0"/>
+    <xacro:property name="max_steering_effort"           value="10.0"/>
     <xacro:property name="max_velocity"                  value="2.0"/>
     <xacro:property name="max_effort"                    value="10.0"/>
@@ -80,8 +80,9 @@
                            h="${chassis_height}"/>
     </link>
+    <!-- No rotation — X is forward, Y is left, Z is up -->
     <joint name="base_to_chassis" type="fixed">
         <parent link="base_link"/>
         <child  link="chassis"/>
-        <origin xyz="0 0 ${wheel_radius + chassis_height/2}" rpy="0 0 3.1416"/>
+        <origin xyz="0 0 ${wheel_radius + chassis_height/2}" rpy="0 0 0"/>
     </joint>
     <!-- ===== WHEEL MACROS ===== -->
@@ -165,5 +166,5 @@
                    upper="${max_steering_angle}"
                    velocity="${max_steering_angular_velocity}"/>
-            <dynamics damping="0.1" friction="0.1"/>
+            <dynamics damping="1.0" friction="0.1"/>
         </joint>
         <joint name="${prefix}_wheel_joint" type="continuous">
@@ -235,5 +236,5 @@
         <parent link="chassis"/>
         <child  link="camera_link"/>
-        <origin xyz="${chassis_length/2 + camera_depth/2} 0 ${chassis_height/2}"/>
+        <origin xyz="${chassis_length/2 + camera_depth/2} 0 0"/>
     </joint>
     <!-- ===== GAZEBO SIMULATION SETUP ===== -->
@@ -244,18 +245,18 @@
     </gazebo>
     <gazebo reference="front_left_wheel_link">
-        <mu1>0.8</mu1>
-        <mu2>0.8</mu2>
+        <mu1>100.0</mu1>
+        <mu2>100.0</mu2>
     </gazebo>
     <gazebo reference="front_right_wheel_link">
-        <mu1>0.8</mu1>
-        <mu2>0.8</mu2>
+        <mu1>100.0</mu1>
+        <mu2>100.0</mu2>
     </gazebo>
     <gazebo reference="rear_left_wheel_link">
-        <mu1>0.8</mu1>
-        <mu2>0.8</mu2>
+        <mu1>100.0</mu1>
+        <mu2>100.0</mu2>
     </gazebo>
     <gazebo reference="rear_right_wheel_link">
-        <mu1>0.8</mu1>
-        <mu2>0.8</mu2>
+        <mu1>100.0</mu1>
+        <mu2>100.0</mu2>
     </gazebo>
     <gazebo reference="lidar_link">

Commit message: LQR controller added

File: src/mr_peterbot_description/urdf/mr_peterbot.urdf.xacro (robot description, xacro)
@@ -17,5 +17,5 @@
     <xacro:property name="max_steering_angular_velocity" value="1.570796"/>
     <xacro:property name="max_steering_effort"           value="10.0"/>
-    <xacro:property name="max_velocity"                  value="2.0"/>
+    <xacro:property name="max_velocity"                  value="0.2"/>
     <xacro:property name="max_effort"                    value="10.0"/>
     <xacro:property name="max_wheel_angular_velocity"    value="${max_velocity / wheel_radius}"/>
@@ -183,5 +183,5 @@
             <child link="${prefix}_wheel_link"/>
             <axis xyz="0 0 1"/>
-            <dynamics damping="0.1" friction="0.1"/>
+            <dynamics damping="0.01" friction="0.01"/>
         </joint>
     </xacro:macro>
@@ -332,4 +332,10 @@
             <render_engine>ogre2</render_engine>
         </plugin>
+        <plugin filename="gz-sim-odometry-publisher-system"
+                name="gz::sim::systems::OdometryPublisher">
+            <odom_frame>odom</odom_frame>
+            <robot_base_frame>base_link</robot_base_frame>
+            <publish_rate>50</publish_rate>
+        </plugin>
     </gazebo>
 </robot>
